File: ATmega328PB-bread-board.kicad_pcb (KiCad board)
At the start: 2 copper layers, 60 x 60 mm, 12 parts, among them J1 Conn_01x17, J2 Conn_01x17, U1 ATmega328PB-MU

Commit message: Update revision to Rev2021.04
Other:
- board text added: "rev2021.04"
- board text removed: "rev2021.03"
Changed lines of the file:
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@@
     (effects (font (size 1 1) (thickness 0.15)))
   )
-  (gr_text rev2021.03 (at 146.35 108.48) (layer F.SilkS)
+  (gr_text rev2021.04 (at 146.35 108.48) (layer F.SilkS)
     (effects (font (size 1 1) (thickness 0.15)))
   )
